File: KiCad/Nanopipetes/DAC_filter.kicad_sch (KiCad schematic)
At the start: 38 parts, among them IC18 OPA4317ID, IC19 OPA4317ID

Commit message: kicad v 1.03
Connections:
- net +5V: no longer IC19.4 (V+)
- net +3.3VDA renamed +3.3VD_ADC
- net +3.3VD_ADC: now also IC19.4 (V+)
Changed lines of the file:
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@@
 			)
 		)
-		(property "Value" "+3.3VDA"
+		(property "Value" "+3.3VD_ADC"
 			(at 207.01 45.466 0)
 			(effects
@@
 			)
 		)
-		(property "Value" "+5V"
+		(property "Value" "+3.3VD_ADC"
 			(at 212.09 115.316 0)
 			(effects
