File: KiCad/Nanopipetes/IV_Converter1.kicad_sch (KiCad schematic)
At the start: 20 parts, among them IC4 OPA827AIDR, IC5 OPA827AIDR, IC6 OPA827AIDR, IC7 OPA827AIDR

Commit message: kicad v 1.03
Parts:
- removed IC4, IC5, IC6, IC7: OPA827AIDR, SamacSys_Parts:SOIC127P600X175-8N, symbol SamacSys_Parts:OPA827AIDR
- added IC4, IC5, IC6, IC7: OPA380AID, Custom:SOIC127P600X175-8N, symbol OPA380AID:OPA380AID
- C27, C28, C29: now not fitted
Connections:
- net +1.25V_VCOM: now also IC4.3 (+IN), IC5.3 (+IN), IC6.3 (+IN), IC7.3 (+IN)
- net +3.3VA_ADC: now also IC4.7 (V+), IC5.7 (V+), IC6.7 (V+), IC7.7 (V+)
- net GND: now also IC4.4 (V-), IC5.4 (V-), IC6.4 (V-), IC7.4 (V-)
- net IN1: now also IC4.2 (-IN)
- net IN2: now also IC6.2 (-IN)
- net IN3: now also IC5.2 (-IN)
- net IN4: now also IC7.2 (-IN)
- net OUT1: now also IC4.6 (OUT)
- net OUT2: now also IC6.6 (OUT)
- net OUT3: now also IC5.6 (OUT)
- net OUT4: now also IC7.6 (OUT)
