File: KiCad/Nanopipetes/IV_Converter2.kicad_sch (KiCad schematic)
At the start: 20 parts, among them IC10 OPA827AIDR, IC11 OPA827AIDR, IC12 OPA827AIDR, IC9 OPA827AIDR

Commit message: kicad v 1.03
Parts:
- removed IC10, IC11, IC12, IC9: OPA827AIDR, SamacSys_Parts:SOIC127P600X175-8N, symbol SamacSys_Parts:OPA827AIDR
- added IC10, IC11, IC12, IC9: OPA380AID, Custom:SOIC127P600X175-8N, symbol OPA380AID:OPA380AID
- C45, C46, C47, C48: now not fitted
Connections:
- net +1.25V_VCOM: now also IC10.3 (+IN), IC11.3 (+IN), IC12.3 (+IN), IC9.3 (+IN)
- net +3.3VA_ADC: now also IC10.7 (V+), IC11.7 (V+), IC12.7 (V+), IC9.7 (V+)
- net GND: now also IC10.4 (V-), IC11.4 (V-), IC12.4 (V-), IC9.4 (V-)
- net IN5: now also IC9.2 (-IN)
- net IN6: now also IC11.2 (-IN)
- net IN7: now also IC10.2 (-IN)
- net IN8: now also IC12.2 (-IN)
- net OUT5: now also IC9.6 (OUT)
- net OUT6: now also IC11.6 (OUT)
- net OUT7: now also IC10.6 (OUT)
- net OUT8: now also IC12.6 (OUT)
