File: KiCad/Nanopipetes/Nanopipetes.kicad_pcb (KiCad board)
At the start: 4 copper layers, 112.8 x 102.2 mm, 298 parts, among them IC1 OPA827AIDR, IC10 OPA827AIDR, IC11 OPA827AIDR, IC12 OPA827AIDR, IC13 AD7383-4BCPZ, IC14 DAC80508ZCRTET, IC15 10M50SCE144C8G, IC16 DEL-DP83867IRPAPT, IC17 M93C46-WMN6TP, IC18 OPA4317ID, IC19 OPA4317ID, IC2 ADR4525ARZ-R7, IC3 TLV70311DBVR, IC4 OPA827AIDR, IC5 OPA827AIDR, IC6 OPA827AIDR, IC7 OPA827AIDR, IC8 AD7383-4BCPZ, IC9 OPA827AIDR, J1 Conn_01x05_Pin, J2 USB_A, J3 Conn_01x03_Pin, J4 Screw_Terminal_01x09, J5 Screw_Terminal_01x09, J6 73099-0, J7 Screw_Terminal_01x02, J8 Conn_01x04_Pin, J9 Conn_02x05_Odd_Even, Q1 MMBT3904, Q2 MMBT3904, T1 WE-RJ45_7499111221A, U1 AMS1117-3.3, U2 AMS1117-1.8, U3 AMS1117-3.3, U4 AMS1117-2.5, U5 AMS1117-3.3, U6 AMS1117-3.3, U9 FT2232HQ, Y1 25MHz, Y2 12MHz

Commit message: kicad v 1.03
Parts:
- removed Y1: 25MHz, Custom:XTAL1140X470X330D1270L391X60N
- added R36: 0, Resistor_SMD:R_0603_1608Metric, F.Cu at (205.9, 58.8)
- C38, C57: value 0.1µF -> 1µF
- IC10, IC11, IC12, IC4, IC5, IC6, IC7, IC9: value OPA827AIDR -> OPA380AID; footprint SamacSys_Parts:SOIC127P600X175-8N -> Custom:SOIC127P600X175-8N
- moved R14 0.44 mm to (124.3, 122.9)
- moved R12 0.32 mm to (124.4, 116.5)
Connections:
- IC10 pad 1: unconnected-(IC10-NC-Pad1) -> (no net)
- IC10 pad 5: unconnected-(IC10-NC-Pad5) -> (no net)
- IC10 pad 8: unconnected-(IC10-NC-Pad8) -> (no net)
- IC11 pad 1: unconnected-(IC11-NC-Pad1) -> (no net)
- IC11 pad 5: unconnected-(IC11-NC-Pad5) -> (no net)
- IC11 pad 8: unconnected-(IC11-NC-Pad8) -> (no net)
- IC12 pad 1: unconnected-(IC12-NC-Pad1) -> (no net)
- IC12 pad 5: unconnected-(IC12-NC-Pad5) -> (no net)
- IC12 pad 8: unconnected-(IC12-NC-Pad8) -> (no net)
- IC18 pad 4: +5V -> +3.3VD_ADC
- IC19 pad 4: +5V -> +3.3VD_ADC
- IC4 pad 1: unconnected-(IC4-NC-Pad1) -> (no net)
- IC4 pad 5: unconnected-(IC4-NC-Pad5) -> (no net)
- IC4 pad 8: unconnected-(IC4-NC-Pad8) -> (no net)
- IC5 pad 1: unconnected-(IC5-NC-Pad1) -> (no net)
- IC5 pad 5: unconnected-(IC5-NC-Pad5) -> (no net)
- IC5 pad 8: unconnected-(IC5-NC-Pad8) -> (no net)
- IC6 pad 1: unconnected-(IC6-NC-Pad1) -> (no net)
- IC6 pad 5: unconnected-(IC6-NC-Pad5) -> (no net)
- IC6 pad 8: unconnected-(IC6-NC-Pad8) -> (no net)
- IC7 pad 1: unconnected-(IC7-NC-Pad1) -> (no net)
- IC7 pad 5: unconnected-(IC7-NC-Pad5) -> (no net)
- IC7 pad 8: unconnected-(IC7-NC-Pad8) -> (no net)
- IC9 pad 1: unconnected-(IC9-NC-Pad1) -> (no net)
- IC9 pad 5: unconnected-(IC9-NC-Pad5) -> (no net)
- IC9 pad 8: unconnected-(IC9-NC-Pad8) -> (no net)
- J2 pad 4: GND -> Net-(J2-GND)
- J2 pad 5: GND -> Net-(J2-GND)
Routing:
- net +3.3VD_ADC: track 135.4 -> 158.5 mm, vias 4 -> 6
- net Net-(J2-GND): track 0.00 -> 18.8 mm
- net GND: track 300.3 -> 286.8 mm
- net Net-(IC16-X_O): track 4.08 -> 15.1 mm
- net Net-(IC16-X_I): track 3.66 -> 10.4 mm
- net +5V: track 35.8 -> 32.8 mm, vias 17 -> 15
- net /Ethernet/Ethernet.MDIO: track 31.4 -> 29.6 mm, vias 2 -> 3
- net /ADC2/IN6: track 48.8 -> 47.8 mm
- net +3.3VD: track 162.1 -> 163.0 mm
- net /DAC/DAC.SDO: track 44.8 -> 43.9 mm
- net +1.1V_ETH: track 127.0 -> 127.6 mm
- net /USB/OSCN: track 11.9 -> 12.4 mm
- net /ADC2/IN5: track 47.6 -> 47.0 mm
