File: KiCad/Nanopipetes/USB.kicad_sch (KiCad schematic)
At the start: 27 parts, among them IC17 M93C46-WMN6TP, J2 USB_A, U9 FT2232HQ, Y2 12MHz

Commit message: kicad v 1.03
Parts:
- R36: footprint (none) -> Resistor_SMD:R_0603_1608Metric
Changed lines of the file:
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@@
 			)
 		)
-		(property "Footprint" ""
+		(property "Footprint" "Resistor_SMD:R_0603_1608Metric"
 			(at 45.212 91.44 90)
 			(effects
